File: PWR_LDO.kicad_sch (KiCad schematic)
At the start: 20 parts, among them U6 TLV75801PDBV, U7 TLV75801PDBV, U8 TLV75801PDBV, U9 TLV75801PDBV

Commit message: layout plan
Parts:
- C21, C22, C23, C24, C25, C26, C27, C28: renamed from C1; footprint (none) -> Capacitor_SMD:C_0603_1608Metric_Pad1.08x0.95mm_HandSolder
- R21, R22, R23, R24, R25, R26, R27, R28: footprint (none) -> Resistor_SMD:R_0603_1608Metric_Pad0.98x0.95mm_HandSolder
