File: space-berry.kicad_pcb (KiCad board)
At the start: 6 copper layers, 0 parts

Commit message: layout plan
Parts:
- added C1: 20uF, Capacitor_SMD:C_1206_3216Metric_Pad1.33x1.80mm_HandSolder, F.Cu at (94.3, 32.7)
- added C10: 44uF, Capacitor_SMD:C_1206_3216Metric_Pad1.33x1.80mm_HandSolder, F.Cu at (105.2, 45.4)
- added C11: 100nF, Capacitor_SMD:C_0603_1608Metric_Pad1.08x0.95mm_HandSolder, F.Cu at (107.5, 44.2)
- added C12: 20uF, Capacitor_SMD:C_1206_3216Metric_Pad1.33x1.80mm_HandSolder, F.Cu at (105.8, 32.8)
- added C13: 44uF, Capacitor_SMD:C_1206_3216Metric_Pad1.33x1.80mm_HandSolder, F.Cu at (70.9, 45.4)
- added C14: 100nF, Capacitor_SMD:C_0603_1608Metric_Pad1.08x0.95mm_HandSolder, F.Cu at (73.2, 44.2)
- added C15: 20uF, Capacitor_SMD:C_1206_3216Metric_Pad1.33x1.80mm_HandSolder, F.Cu at (71.5, 32.8)
- added C16: 44uF, Capacitor_SMD:C_1206_3216Metric_Pad1.33x1.80mm_HandSolder, F.Cu at (128.2, 45.5)
- added C17: 100nF, Capacitor_SMD:C_0603_1608Metric_Pad1.08x0.95mm_HandSolder, F.Cu at (130.5, 44.3)
- added C18: 20uF, Capacitor_SMD:C_1206_3216Metric_Pad1.33x1.80mm_HandSolder, F.Cu at (128.8, 32.9)
- added C2: 44uF, Capacitor_SMD:C_1206_3216Metric_Pad1.33x1.80mm_HandSolder, F.Cu at (93.7, 45.3)
- added C21: 10uf, Capacitor_SMD:C_0603_1608Metric_Pad1.08x0.95mm_HandSolder, F.Cu at (136.3, 46.8)
- added C22: 10uf, Capacitor_SMD:C_0603_1608Metric_Pad1.08x0.95mm_HandSolder, F.Cu at (139.1, 51.8)
- added C23: 10uf, Capacitor_SMD:C_0603_1608Metric_Pad1.08x0.95mm_HandSolder, F.Cu at (152.0, 46.8)
- added C24: 10uf, Capacitor_SMD:C_0603_1608Metric_Pad1.08x0.95mm_HandSolder, F.Cu at (154.7, 51.8)
- added C25: 10uf, Capacitor_SMD:C_0603_1608Metric_Pad1.08x0.95mm_HandSolder, F.Cu at (144.2, 46.8)
- added C26: 10uf, Capacitor_SMD:C_0603_1608Metric_Pad1.08x0.95mm_HandSolder, F.Cu at (147.0, 51.7)
- added C27: 10uf, Capacitor_SMD:C_0603_1608Metric_Pad1.08x0.95mm_HandSolder, F.Cu at (112.1, 55.6)
- added C28: 10uf, Capacitor_SMD:C_0603_1608Metric_Pad1.08x0.95mm_HandSolder, F.Cu at (117.1, 52.9)
- added C3: 100nF, Capacitor_SMD:C_0603_1608Metric_Pad1.08x0.95mm_HandSolder, F.Cu at (96.0, 44.1)
- added C4: 44uF, Capacitor_SMD:C_1206_3216Metric_Pad1.33x1.80mm_HandSolder, F.Cu at (82.2, 45.4)
- added C5: 100nF, Capacitor_SMD:C_0603_1608Metric_Pad1.08x0.95mm_HandSolder, F.Cu at (84.5, 44.2)
- added C6: 20uF, Capacitor_SMD:C_1206_3216Metric_Pad1.33x1.80mm_HandSolder, F.Cu at (82.8, 32.8)
- added C7: 44uF, Capacitor_SMD:C_1206_3216Metric_Pad1.33x1.80mm_HandSolder, F.Cu at (116.8, 45.4)
- added C8: 100nF, Capacitor_SMD:C_0603_1608Metric_Pad1.08x0.95mm_HandSolder, F.Cu at (119.1, 44.2)
- added C9: 20uF, Capacitor_SMD:C_1206_3216Metric_Pad1.33x1.80mm_HandSolder, F.Cu at (117.4, 32.8)
- added D1: LED, LED_SMD:LED_0603_1608Metric_Pad1.05x0.95mm_HandSolder, F.Cu at (62.0, 61.0)
- added F1: Fuse, Fuse:Fuse_1210_3225Metric_Pad1.42x2.65mm_HandSolder, F.Cu at (135.8, 38.8)
- added Q1: SiS415DNT, Package_SO:Vishay_PowerPAK_1212-8_Single, F.Cu at (135.6, 33.0)
- added Q2: TSM2302CX, Package_TO_SOT_SMD:SOT-23, F.Cu at (62.0, 50.0)
- added R1: R adj, Resistor_SMD:R_0603_1608Metric_Pad0.98x0.95mm_HandSolder, F.Cu at (90.6, 43.6)
- added R10: 1k opt, Resistor_SMD:R_0603_1608Metric_Pad0.98x0.95mm_HandSolder, F.Cu at (107.5, 36.8)
- added R11: 20K opt, Resistor_SMD:R_0603_1608Metric_Pad0.98x0.95mm_HandSolder, F.Cu at (107.5, 40.5)
- added R12: R adj, Resistor_SMD:R_0603_1608Metric_Pad0.98x0.95mm_HandSolder, F.Cu at (102.1, 43.7)
- added R13: 1k opt, Resistor_SMD:R_0603_1608Metric_Pad0.98x0.95mm_HandSolder, F.Cu at (73.2, 36.8)
- added R14: 20K opt, Resistor_SMD:R_0603_1608Metric_Pad0.98x0.95mm_HandSolder, F.Cu at (73.2, 40.5)
- added R15: R adj, Resistor_SMD:R_0603_1608Metric_Pad0.98x0.95mm_HandSolder, F.Cu at (67.8, 43.7)
- added R16: 1k opt, Resistor_SMD:R_0603_1608Metric_Pad0.98x0.95mm_HandSolder, F.Cu at (130.5, 36.9)
- added R17: 20K opt, Resistor_SMD:R_0603_1608Metric_Pad0.98x0.95mm_HandSolder, F.Cu at (130.5, 40.6)
- added R18: R adj, Resistor_SMD:R_0603_1608Metric_Pad0.98x0.95mm_HandSolder, F.Cu at (125.1, 43.8)
- added R2: 20K opt, Resistor_SMD:R_0603_1608Metric_Pad0.98x0.95mm_HandSolder, F.Cu at (96.0, 40.4)
- added R21: R, Resistor_SMD:R_0603_1608Metric_Pad0.98x0.95mm_HandSolder, F.Cu at (139.1, 48.0)
- added R22: R, Resistor_SMD:R_0603_1608Metric_Pad0.98x0.95mm_HandSolder, F.Cu at (136.2, 53.2)
- added R23: R, Resistor_SMD:R_0603_1608Metric_Pad0.98x0.95mm_HandSolder, F.Cu at (152.0, 53.2)
- added R24: R, Resistor_SMD:R_0603_1608Metric_Pad0.98x0.95mm_HandSolder, F.Cu at (154.7, 48.0)
- added R25: R, Resistor_SMD:R_0603_1608Metric_Pad0.98x0.95mm_HandSolder, F.Cu at (147.0, 48.0)
- added R26: R, Resistor_SMD:R_0603_1608Metric_Pad0.98x0.95mm_HandSolder, F.Cu at (144.2, 53.2)
- added R27: R, Resistor_SMD:R_0603_1608Metric_Pad0.98x0.95mm_HandSolder, F.Cu at (118.3, 55.6)
- added R28: R, Resistor_SMD:R_0603_1608Metric_Pad0.98x0.95mm_HandSolder, F.Cu at (113.3, 52.9)
- added R29: 10, Resistor_SMD:R_0603_1608Metric_Pad0.98x0.95mm_HandSolder, F.Cu at (62.0, 59.0)
- added R3: 1k opt, Resistor_SMD:R_0603_1608Metric_Pad0.98x0.95mm_HandSolder, F.Cu at (96.0, 36.7)
- added R30: 10K, Resistor_SMD:R_0603_1608Metric_Pad0.98x0.95mm_HandSolder, F.Cu at (62.0, 57.0)
- added R31: 10K, Resistor_SMD:R_0603_1608Metric_Pad0.98x0.95mm_HandSolder, F.Cu at (62.0, 55.1)
- added R32: 10K, Resistor_SMD:R_0603_1608Metric_Pad0.98x0.95mm_HandSolder, F.Cu at (62.0, 53.0)
- added R4: 1k opt, Resistor_SMD:R_0603_1608Metric_Pad0.98x0.95mm_HandSolder, F.Cu at (84.5, 36.8)
- added R5: 20K opt, Resistor_SMD:R_0603_1608Metric_Pad0.98x0.95mm_HandSolder, F.Cu at (84.5, 40.5)
- added R6: R adj, Resistor_SMD:R_0603_1608Metric_Pad0.98x0.95mm_HandSolder, F.Cu at (79.1, 43.7)
- added R7: 1k opt, Resistor_SMD:R_0603_1608Metric_Pad0.98x0.95mm_HandSolder, F.Cu at (119.1, 36.8)
- added R8: 20K opt, Resistor_SMD:R_0603_1608Metric_Pad0.98x0.95mm_HandSolder, F.Cu at (119.1, 40.5)
- added R9: R adj, Resistor_SMD:R_0603_1608Metric_Pad0.98x0.95mm_HandSolder, F.Cu at (113.7, 43.7)
- added REF**: MountingHole_3.2mm_M3_Pad_Via, MountingHole:MountingHole_3.2mm_M3_Pad_Via, F.Cu at (155.5, 124.5)
- added REF**: BarrelJack_CUI_PJ-063AH_Horizontal, Connector_BarrelJack:BarrelJack_CUI_PJ-063AH_Horizontal, F.Cu at (145.0, 40.2)
- added REF**: RJ45_Abracon_ARJP11A-MA_Horizontal, Connector_RJ:RJ45_Abracon_ARJP11A-MA_Horizontal, F.Cu at (69.8, 109.0)
- added REF**: USB_C_Receptacle_GCT_USB4105-xx-A_16P_TopMnt_Horizontal, Connector_USB:USB_C_Receptacle_GCT_USB4105-xx-A_16P_TopMnt_Horizontal, F.Cu at (110.9, 124.5)
- added REF**: FBGA96X16_7P5X13P3_SAM, lib:FBGA96X16_7P5X13P3_SAM, F.Cu at (134.0, 88.9)
- added REF**: MountingHole_3.2mm_M3_Pad_Via, MountingHole:MountingHole_3.2mm_M3_Pad_Via, F.Cu at (62.8, 124.5)
- added REF**: microSD_HC_Molex_47219-2001, Connector_Card:microSD_HC_Molex_47219-2001, F.Cu at (94.4, 120.8)
- added REF**: HDMI_A_Molex_208658-1001_Horizontal, Connector_HDMI:HDMI_A_Molex_208658-1001_Horizontal, F.Cu at (141.5, 121.1)
- added REF**: PinHeader_2x08_P2.54mm_Vertical_SMD, Connector_PinHeader_2.54mm:PinHeader_2x08_P2.54mm_Vertical_SMD, F.Cu at (152.6, 69.7)
- added REF**: USB_C_Receptacle_GCT_USB4105-xx-A_16P_TopMnt_Horizontal, Connector_USB:USB_C_Receptacle_GCT_USB4105-xx-A_16P_TopMnt_Horizontal, F.Cu at (124.1, 124.5)
- added REF**: MountingHole_3.2mm_M3_Pad_Via, MountingHole:MountingHole_3.2mm_M3_Pad_Via, F.Cu at (155.6, 31.8)
- added REF**: SW_DIP_SPSTx04_Slide_KingTek_DSHP04TJ_W5.25mm_P1.27mm_JPin, Button_Switch_SMD:SW_DIP_SPSTx04_Slide_KingTek_DSHP04TJ_W5.25mm_P1.27mm_JPin, F.Cu at (153.0, 86.3)
- added REF**: MountingHole_3.2mm_M3_Pad_Via, MountingHole:MountingHole_3.2mm_M3_Pad_Via, F.Cu at (62.8, 31.8)
- added TP1: PG, TestPoint:TestPoint_Pad_D1.0mm, F.Cu at (88.5, 46.9)
- added TP10: Vout, TestPoint:TestPoint_Pad_D1.0mm, F.Cu at (107.4, 47.0)
- added TP11: PG, TestPoint:TestPoint_Pad_D1.0mm, F.Cu at (100.0, 47.0)
- added TP12: EN, TestPoint:TestPoint_Pad_D1.0mm, F.Cu at (102.5, 47.0)
- added TP13: Vout, TestPoint:TestPoint_Pad_D1.0mm, F.Cu at (73.1, 47.0)
- added TP14: PG, TestPoint:TestPoint_Pad_D1.0mm, F.Cu at (65.7, 47.0)
- added TP15: EN, TestPoint:TestPoint_Pad_D1.0mm, F.Cu at (68.2, 47.0)
- added TP16: Vout, TestPoint:TestPoint_Pad_D1.0mm, F.Cu at (130.4, 47.1)
- added TP17: PG, TestPoint:TestPoint_Pad_D1.0mm, F.Cu at (123.0, 47.1)
- added TP18: EN, TestPoint:TestPoint_Pad_D1.0mm, F.Cu at (125.5, 47.1)
- added TP2: EN, TestPoint:TestPoint_Pad_D1.0mm, F.Cu at (91.0, 46.9)
- added TP3: Vout, TestPoint:TestPoint_Pad_D1.0mm, F.Cu at (95.9, 46.9)
- added TP4: Vout, TestPoint:TestPoint_Pad_D1.0mm, F.Cu at (84.4, 47.0)
- added TP5: PG, TestPoint:TestPoint_Pad_D1.0mm, F.Cu at (77.0, 47.0)
- added TP6: EN, TestPoint:TestPoint_Pad_D1.0mm, F.Cu at (79.5, 47.0)
- added TP7: Vout, TestPoint:TestPoint_Pad_D1.0mm, F.Cu at (119.0, 47.0)
- added TP8: PG, TestPoint:TestPoint_Pad_D1.0mm, F.Cu at (111.6, 47.0)
- added TP9: EN, TestPoint:TestPoint_Pad_D1.0mm, F.Cu at (114.1, 47.0)
- added U1: ~, lib:NAM12S06-D, F.Cu at (90.8, 38.4)
- added U10: ~, lib:NAM12S06-D, F.Cu at (125.2, 38.7)
- added U12: K4A8G165WC-BCTD, lib:FBGA96X16_7P5X13P3_SAM, F.Cu at (134.0, 71.5)
- added U13: XCZU15EG-2FFVB1156E, lib:FFVB1156_XIL-L, F.Cu at (109.0, 78.0)
- added U2: ~, lib:NAM12S06-D, F.Cu at (79.2, 38.5)
- added U3: ~, lib:NAM12S06-D, F.Cu at (113.8, 38.5)
- added U4: ~, lib:NAM12S06-D, F.Cu at (102.2, 38.5)
- added U5: ~, lib:NAM12S06-D, F.Cu at (68.0, 38.5)
- added U6: TLV75801PDBV, Package_TO_SOT_SMD:SOT-23-5, F.Cu at (152.0, 50.0)
- added U7: TLV75801PDBV, Package_TO_SOT_SMD:SOT-23-5, F.Cu at (144.2, 50.0)
- added U8: TLV75801PDBV, Package_TO_SOT_SMD:SOT-23-5, F.Cu at (136.2, 50.0)
- added U9: TLV75801PDBV, Package_TO_SOT_SMD:SOT-23-5, F.Cu at (115.3, 55.6)
Routing:
- net VCC: track 0.00 -> 101.9 mm
- net Net-(U4-EN): track 0.00 -> 31.4 mm, vias 0 -> 4
- net Net-(U1-EN): track 0.00 -> 31.4 mm, vias 0 -> 4
- net Net-(U3-EN): track 0.00 -> 31.4 mm, vias 0 -> 4
- net Net-(U10-EN): track 0.00 -> 31.4 mm, vias 0 -> 4
- net Net-(U2-EN): track 0.00 -> 31.4 mm, vias 0 -> 4
- net Net-(U3-PG): track 0.00 -> 31.0 mm, vias 0 -> 4
- net Net-(U2-PG): track 0.00 -> 31.0 mm, vias 0 -> 4
- net Net-(U4-PG): track 0.00 -> 31.0 mm, vias 0 -> 4
- net Net-(U10-PG): track 0.00 -> 31.0 mm, vias 0 -> 4
- net Net-(U1-PG): track 0.00 -> 31.0 mm, vias 0 -> 4
- net DDR_PAR: track 0.00 -> 27.5 mm, vias 0 -> 2
- net DDR_RES: track 0.00 -> 23.7 mm, vias 0 -> 2
- net GND: track 0.00 -> 20.0 mm, vias 0 -> 22
- net DDR_ALTER: track 0.00 -> 19.8 mm, vias 0 -> 2
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- added copper zone on F.Cu, net Net-(C10-Pad1)
- added copper zone on F.Cu, net Net-(C13-Pad1)
- added copper zone on F.Cu, net Net-(C16-Pad1)
- added copper zone on F.Cu, net Net-(C2-Pad1)
- added copper zone on F.Cu, net Net-(C4-Pad1)
- added copper zone on F.Cu, net Net-(C7-Pad1)
- added copper zone on F.Cu, net VCC
