File: space-berry.kicad_sch (KiCad schematic)
At the start: 0 parts

Commit message: layout plan
Other:
- removed sheet PWR_0V85
- removed sheet PWR_1V2
- removed sheet PWR_1V8
- removed sheet PWR_3V3
- removed sheet PWR_3V3_AUX
- removed sheet PWR_5V0
- added sheet PS_DDR4 (PS_DDR4.kicad_sch)
- added sheet PS_DDR4_BANK (PS_DDR4_BANK.kicad_sch)
- added sheet PS_DDR4_PWR (PS_DDR4_PWR.kicad_sch)
- added sheet PWR_template (PWR_template.kicad_sch)
- added sheet PWR_template1 (PWR_template.kicad_sch)
- added sheet PWR_template2 (PWR_template.kicad_sch)
- added sheet PWR_template3 (PWR_template.kicad_sch)
- added sheet PWR_template4 (PWR_template.kicad_sch)
- added sheet PWR_template5 (PWR_template.kicad_sch)
Changed lines of the file:
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@@
 (kicad_sch (version 20230121) (generator eeschema)
   (paper "A4")
-  (sheet (at 38.1 139.7) (size 25.4 12.7) (fields_autoplaced)
+  (sheet (at 38.1 38.1) (size 25.4 12.7) (fields_autoplaced)
     (stroke (width 0.1524) (type solid))
     (fill (color 0 0 0 0.0000))
-    (property "Sheetname" "PWR_3V3_AUX" (at 38.1 138.9884 0)
+    (property "Sheetname" "PWR_template" (at 38.1 37.3884 0)
       (effects (font (size 1.27 1.27)) (justify left bottom))
     )
-    (property "Sheetfile" "PWR_3V3_AUX.kicad_sch" (at 38.1 152.9846 0)
-      (effects (font (size 1.27 1.27)) (justify left top))
-    )
-    (instances
-      (project "space-berry"
-        (path "/93269f17-932e-47e4-8e03-ce157f57b85f" (page "6"))
-      )
-    )
-  )
-  (sheet (at 38.1 63.5) (size 25.4 12.7) (fields_autoplaced)
-    (stroke (width 0.1524) (type solid))
-    (fill (color 0 0 0 0.0000))
-    (property "Sheetname" "PWR_1V2" (at 38.1 62.7884 0)
-      (effects (font (size 1.27 1.27)) (justify left bottom))
-    )
-    (property "Sheetfile" "PWR_1V2.kicad_sch" (at 38.1 76.7846 0)
+    (property "Sheetfile" "PWR_template.kicad_sch" (at 38.1 51.3846 0)
       (effects (font (size 1.27 1.27)) (justify left top))
     )
@@
     (stroke (width 0.1524) (type solid))
     (fill (color 0 0 0 0.0000))
-    (property "Sheetname" "PWR_3V3" (at 38.1 113.5884 0)
+    (property "Sheetname" "PWR_template3" (at 38.1 113.5884 0)
       (effects (font (size 1.27 1.27)) (justify left bottom))
     )
-    (property "Sheetfile" "PWR_3V3.kicad_sch" (at 38.1 127.5846 0)
+    (property "Sheetfile" "PWR_template.kicad_sch" (at 38.1 127.5846 0)
       (effects (font (size 1.27 1.27)) (justify left top))
     )
     (instances
       (project "space-berry"
-        (path "/93269f17-932e-47e4-8e03-ce157f57b85f" (page "5"))
-      )
-    )
-  )
-  (sheet (at 38.1 38.1) (size 25.4 12.7) (fields_autoplaced)
-    (stroke (width 0.1524) (type solid))
-    (fill (color 0 0 0 0.0000))
-    (property "Sheetname" "PWR_0V85" (at 38.1 37.3884 0)
-      (effects (font (size 1.27 1.27)) (justify left bottom))
-    )
-    (property "Sheetfile" "PWR_0V85.kicad_sch" (at 38.1 51.3846 0)
-      (effects (font (size 1.27 1.27)) (justify left top))
-    )
-    (instances
-      (project "space-berry"
-        (path "/93269f17-932e-47e4-8e03-ce157f57b85f" (page "2"))
+        (path "/93269f17-932e-47e4-8e03-ce157f57b85f" (page "6"))
       )
     )
@@
     (stroke (width 0.1524) (type solid))
     (fill (color 0 0 0 0.0000))
-    (property "Sheetname" "PWR_LDO" (at 38.1 164.3884 0)
+    (property "Sheetname" "PWR_template5" (at 38.1 164.3884 0)
       (effects (font (size 1.27 1.27)) (justify left bottom))
     )
-    (property "Sheetfile" "PWR_LDO.kicad_sch" (at 38.1 178.3846 0)
+    (property "Sheetfile" "PWR_template.kicad_sch" (at 38.1 178.3846 0)
+      (effects (font (size 1.27 1.27)) (justify left top))
+    )
+    (instances
+      (project "space-berry"
+        (path "/93269f17-932e-47e4-8e03-ce157f57b85f" (page "9"))
+      )
+    )
+  )
+  (sheet (at 76.2 63.5) (size 25.4 12.7) (fields_autoplaced)
+    (stroke (width 0.1524) (type solid))
+    (fill (color 0 0 0 0.0000))
+    (property "Sheetname" "PWR_LDO" (at 76.2 62.7884 0)
+      (effects (font (size 1.27 1.27)) (justify left bottom))
+    )
+    (property "Sheetfile" "PWR_LDO.kicad_sch" (at 76.2 76.7846 0)
       (effects (font (size 1.27 1.27)) (justify left top))
     )
@@
     )
   )
-  (sheet (at 76.2 63.5) (size 25.4 12.7) (fields_autoplaced)
+  (sheet (at 114.3 38.1) (size 25.4 12.7) (fields_autoplaced)
     (stroke (width 0.1524) (type solid))
     (fill (color 0 0 0 0.0000))
-    (property "Sheetname" "PWR_5V0" (at 76.2 62.7884 0)
+    (property "Sheetname" "PS_DDR4" (at 114.3 37.3884 0)
       (effects (font (size 1.27 1.27)) (justify left bottom))
     )
-    (property "Sheetfile" "PWR_5V0.kicad_sch" (at 76.2 76.7846 0)
+    (property "Sheetfile" "PS_DDR4.kicad_sch" (at 114.3 51.3846 0)
+      (effects (font (size 1.27 1.27)) (justify left top))
+    )
+    (instances
+      (project "space-berry"
+        (path "/93269f17-932e-47e4-8e03-ce157f57b85f" (page "10"))
+      )
+    )
+  )
+  (sheet (at 38.1 63.5) (size 25.4 12.7) (fields_autoplaced)
+    (stroke (width 0.1524) (type solid))
+    (fill (color 0 0 0 0.0000))
+    (property "Sheetname" "PWR_template1" (at 38.1 62.7884 0)
+      (effects (font (size 1.27 1.27)) (justify left bottom))
+    )
+    (property "Sheetfile" "PWR_template.kicad_sch" (at 38.1 76.7846 0)
+      (effects (font (size 1.27 1.27)) (justify left top))
+    )
+    (instances
+      (project "space-berry"
+        (path "/93269f17-932e-47e4-8e03-ce157f57b85f" (page "4"))
+      )
+    )
+  )
+  (sheet (at 38.1 139.7) (size 25.4 12.7) (fields_autoplaced)
+    (stroke (width 0.1524) (type solid))
+    (fill (color 0 0 0 0.0000))
+    (property "Sheetname" "PWR_template4" (at 38.1 138.9884 0)
+      (effects (font (size 1.27 1.27)) (justify left bottom))
+    )
+    (property "Sheetfile" "PWR_template.kicad_sch" (at 38.1 152.9846 0)
       (effects (font (size 1.27 1.27)) (justify left top))
     )
@@
       (project "space-berry"
         (path "/93269f17-932e-47e4-8e03-ce157f57b85f" (page "7"))
-      )
-    )
-  )
-  (sheet (at 38.1 88.9) (size 25.4 12.7) (fields_autoplaced)
-    (stroke (width 0.1524) (type solid))
-    (fill (color 0 0 0 0.0000))
-    (property "Sheetname" "PWR_1V8" (at 38.1 88.1884 0)
-      (effects (font (size 1.27 1.27)) (justify left bottom))
-    )
-    (property "Sheetfile" "PWR_1V8.kicad_sch" (at 38.1 102.1846 0)
-      (effects (font (size 1.27 1.27)) (justify left top))
-    )
-    (instances
-      (project "space-berry"
-        (path "/93269f17-932e-47e4-8e03-ce157f57b85f" (page "4"))
       )
     )
@@
     (instances
       (project "space-berry"
-        (path "/93269f17-932e-47e4-8e03-ce157f57b85f" (page "9"))
+        (path "/93269f17-932e-47e4-8e03-ce157f57b85f" (page "2"))
       )
     )
+  )
+  (sheet (at 114.3 88.9) (size 25.4 12.7) (fields_autoplaced)
+    (stroke (width 0.1524) (type solid))
+    (fill (color 0 0 0 0.0000))
+    (property "Sheetname" "PS_DDR4_BANK" (at 114.3 88.1884 0)
+      (effects (font (size 1.27 1.27)) (justify left bottom))
+    )
+    (property "Sheetfile" "PS_DDR4_BANK.kicad_sch" (at 114.3 102.1846 0)
+      (effects (font (size 1.27 1.27)) (justify left top))
+    )
+    (instances
+      (project "space-berry"
+        (path "/93269f17-932e-47e4-8e03-ce157f57b85f" (page "12"))
+      )
+    )
+  )
+  (sheet (at 38.1 88.9) (size 25.4 12.7) (fields_autoplaced)
+    (stroke (width 0.1524) (type solid))
+    (fill (color 0 0 0 0.0000))
+    (property "Sheetname" "PWR_template2" (at 38.1 88.1884 0)
+      (effects (font (size 1.27 1.27)) (justify left bottom))
+    )
+    (property "Sheetfile" "PWR_template.kicad_sch" (at 38.1 102.1846 0)
+      (effects (font (size 1.27 1.27)) (justify left top))
+    )
+    (instances
+      (project "space-berry"
+        (path "/93269f17-932e-47e4-8e03-ce157f57b85f" (page "5"))
+      )
+    )
+  )
+  (sheet (at 114.3 63.5) (size 25.4 12.7) (fields_autoplaced)
+    (stroke (width 0.1524) (type solid))
+    (fill (color 0 0 0 0.0000))
+    (property "Sheetname" "PS_DDR4_PWR" (at 114.3 62.7884 0)
+      (effects (font (size 1.27 1.27)) (justify left bottom))
+    )
+    (property "Sheetfile" "PS_DDR4_PWR.kicad_sch" (at 114.3 76.7846 0)
+      (effects (font (size 1.27 1.27)) (justify left top))
+    )
+    (property "Field2" "" (at 114.3 63.5 0)
+      (effects (font (size 1.27 1.27)) hide)
+    )
+    (instances
+      (project "space-berry"
+        (path "/93269f17-932e-47e4-8e03-ce157f57b85f" (page "11"))
+      )
+    )
