File: Zynq_GND.kicad_sch (KiCad schematic)
At the start: 1 part, among them U13 XCZU15EG-2FFVB1156E

Commit message: Stuff
Parts:
- U13: footprint FFVB1156_XIL -> lib:FFVB1156_XIL-L
Changed lines of the file:
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@@
       (effects (font (size 1.524 1.524)) (justify left))
     )
-    (property "Footprint" "FFVB1156_XIL" (at 227.33 111.76 0)
+    (property "Footprint" "lib:FFVB1156_XIL-L" (at 227.33 111.76 0)
       (effects (font (size 1.27 1.27) italic) hide)
     )
@@
       (effects (font (size 1.524 1.524)) (justify left))
     )
-    (property "Footprint" "FFVB1156_XIL" (at 21.59 20.32 0)
+    (property "Footprint" "lib:FFVB1156_XIL-L" (at 21.59 20.32 0)
       (effects (font (size 1.27 1.27) italic) hide)
     )
@@
       (effects (font (size 1.524 1.524)) (justify left))
     )
-    (property "Footprint" "FFVB1156_XIL" (at 102.87 20.32 0)
+    (property "Footprint" "lib:FFVB1156_XIL-L" (at 102.87 20.32 0)
       (effects (font (size 1.27 1.27) italic) hide)
     )
@@
       (effects (font (size 1.524 1.524)) (justify left))
     )
-    (property "Footprint" "FFVB1156_XIL" (at 143.51 20.32 0)
+    (property "Footprint" "lib:FFVB1156_XIL-L" (at 143.51 20.32 0)
       (effects (font (size 1.27 1.27) italic) hide)
     )
@@
       (effects (font (size 1.524 1.524)) (justify left))
     )
-    (property "Footprint" "FFVB1156_XIL" (at 185.42 20.32 0)
+    (property "Footprint" "lib:FFVB1156_XIL-L" (at 185.42 20.32 0)
       (effects (font (size 1.27 1.27) italic) hide)
     )
@@
       (effects (font (size 1.524 1.524)) (justify left))
     )
-    (property "Footprint" "FFVB1156_XIL" (at 64.77 20.32 0)
+    (property "Footprint" "lib:FFVB1156_XIL-L" (at 64.77 20.32 0)
       (effects (font (size 1.27 1.27) italic) hide)
     )
