File: PWR_3.kicad_sch (KiCad schematic)
At the start: 10 parts

Commit message: DDR4 finish
Connections:
- net 1V2: now reaches C2.1, C3.1, TP3.1, U1.17 (VOUT), U1.18 (VOUT), U1.20 (VOUT), U1.21 (VOUT)
Changed lines of the file:
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@@
   (junction (at 116.84 76.2) (diameter 0) (color 0 0 0 0)
+  )
+  (junction (at 173.99 76.2) (diameter 0) (color 0 0 0 0)
   )
   (junction (at 134.62 134.62) (diameter 0) (color 0 0 0 0)
@@
   )
   (wire (pts (xy 152.4 134.62) (xy 152.4 121.92))
+    (stroke (width 0) (type default))
+  )
+  (wire (pts (xy 173.99 76.2) (xy 175.26 76.2))
     (stroke (width 0) (type default))
   )
@@
     )
   )
+  (global_label "1V2" (shape input) (at 175.26 76.2 0) (fields_autoplaced)
+    (effects (font (size 1.27 1.27)) (justify left))
+    (property "Intersheetrefs" "${INTERSHEET_REFS}" (at 181.6734 76.2 0)
+      (effects (font (size 1.27 1.27)) (justify left) hide)
+    )
+  )
