File: PWR_4.kicad_sch (KiCad schematic)
At the start: 10 parts

Commit message: DDR4 finish
Changed lines of the file:
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@@
+    )
+  )
+  (global_label "2V5_LDO" (shape input) (at 179.07 76.2 0) (fields_autoplaced)
+    (effects (font (size 1.27 1.27)) (justify left))
+    (property "Intersheetrefs" "${INTERSHEET_REFS}" (at 190.0796 76.2 0)
+      (effects (font (size 1.27 1.27)) (justify left) hide)
     )
   )
