File: USB_3.kicad_sch (KiCad schematic)
At the start: 1 part, among them J1 USB_C_Receptacle

Commit message: usb and stuff
Parts:
- added U15: USB3300-EZK, Package_DFN_QFN:QFN-32-1EP_5x5mm_P0.5mm_EP3.45x3.45mm, symbol Interface_USB:USB3300-EZK
Changed lines of the file:
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@@
+    )
+  )
+  (symbol (lib_id "Interface_USB:USB3300-EZK") (at 199.39 96.52 0) (unit 1)
+    (in_bom yes) (on_board yes) (dnp no) (fields_autoplaced)
+    (property "Reference" "U15" (at 203.8859 123.19 0)
+      (effects (font (size 1.27 1.27)) (justify left))
+    )
+    (property "Value" "USB3300-EZK" (at 203.8859 125.73 0)
+      (effects (font (size 1.27 1.27)) (justify left))
+    )
+    (property "Footprint" "Package_DFN_QFN:QFN-32-1EP_5x5mm_P0.5mm_EP3.45x3.45mm" (at 232.41 128.27 0)
+      (effects (font (size 1.27 1.27)) hide)
+    )
+    (property "Datasheet" "http://ww1.microchip.com/downloads/en/DeviceDoc/00001783C.pdf" (at 199.39 96.52 0)
+      (effects (font (size 1.27 1.27)) hide)
+    )
+    (pin "1")
+    (pin "10")
+    (pin "11")
+    (pin "12")
+    (pin "13")
+    (pin "14")
+    (pin "15")
+    (pin "16")
+    (pin "17")
+    (pin "18")
+    (pin "19")
+    (pin "2")
+    (pin "20")
+    (pin "21")
+    (pin "22")
+    (pin "23")
+    (pin "24")
+    (pin "25")
+    (pin "26")
+    (pin "27")
+    (pin "28")
+    (pin "29")
+    (pin "3")
+    (pin "30")
+    (pin "31")
+    (pin "32")
+    (pin "33")
+    (pin "4")
+    (pin "5")
+    (pin "6")
+    (pin "7")
+    (pin "8")
+    (pin "9")
+    (instances
+      (project "space-berry"
+        (path "/93269f17-932e-47e4-8e03-ce157f57b85f/2166ed60-c589-413b-a298-140af16eae77"
+          (reference "U15") (unit 1)
+        )
+        (path "/93269f17-932e-47e4-8e03-ce157f57b85f/1e39a03a-1a0f-461d-8eae-706bef06b5a3"
+          (reference "U16") (unit 1)
+        )
+      )
     )
   )
