File: USB_2.kicad_sch (KiCad schematic)
At the start: 14 parts, among them J3 USB_C_Receptacle_USB2.0, U15 USB3300-EZK, X1 ECS-2520MV-xxx-xx

Commit message: stuff
Parts:
- removed J3: USB_C_Receptacle_USB2.0, Connector_USB:USB_C_Receptacle_G-Switch_GT-USB-7010ASV, symbol Connector:USB_C_Receptacle_USB2.0
Changed lines of the file:
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@@
   (junction (at 236.22 41.91) (diameter 0) (color 0 0 0 0)
   )
-  (junction (at 118.11 69.85) (diameter 0) (color 0 0 0 0)
-  )
   (junction (at 107.95 128.27) (diameter 0) (color 0 0 0 0)
   )
@@
   (junction (at 107.95 109.22) (diameter 0) (color 0 0 0 0)
   )
-  (junction (at 118.11 72.39) (diameter 0) (color 0 0 0 0)
-  )
   (junction (at 236.22 29.21) (diameter 0) (color 0 0 0 0)
   )
   (junction (at 92.71 109.22) (diameter 0) (color 0 0 0 0)
-  )
-  (junction (at 96.52 95.25) (diameter 0) (color 0 0 0 0)
   )
   (junction (at 193.04 67.31) (diameter 0) (color 0 0 0 0)
@@
     (stroke (width 0) (type default))
   )
-  (wire (pts (xy 92.71 95.25) (xy 96.52 95.25))
-    (stroke (width 0) (type default))
-  )
-  (wire (pts (xy 115.57 72.39) (xy 118.11 72.39))
-    (stroke (width 0) (type default))
-  )
   (wire (pts (xy 231.14 41.91) (xy 231.14 43.18))
     (stroke (width 0) (type default))
@@
     (stroke (width 0) (type default))
   )
-  (wire (pts (xy 118.11 69.85) (xy 115.57 69.85))
-    (stroke (width 0) (type default))
-  )
   (wire (pts (xy 240.03 73.66) (xy 240.03 76.2))
     (stroke (width 0) (type default))
@@
     (stroke (width 0) (type default))
   )
-  (wire (pts (xy 92.71 92.71) (xy 92.71 95.25))
-    (stroke (width 0) (type default))
-  )
   (wire (pts (xy 236.22 29.21) (xy 247.65 29.21))
     (stroke (width 0) (type default))
@@
     (stroke (width 0) (type default))
   )
-  (wire (pts (xy 100.33 95.25) (xy 100.33 92.71))
-    (stroke (width 0) (type default))
-  )
   (wire (pts (xy 227.33 63.5) (xy 240.03 63.5))
     (stroke (width 0) (type default))
@@
     (stroke (width 0) (type default))
   )
-  (wire (pts (xy 96.52 95.25) (xy 100.33 95.25))
-    (stroke (width 0) (type default))
-  )
   (wire (pts (xy 224.79 39.37) (xy 224.79 41.91))
     (stroke (width 0) (type default))
   )
-  (wire (pts (xy 96.52 95.25) (xy 96.52 96.52))
-    (stroke (width 0) (type default))
-  )
   (wire (pts (xy 115.57 54.61) (xy 128.27 54.61))
     (stroke (width 0) (type default))
@@
     (stroke (width 0) (type default))
   )
-  (wire (pts (xy 115.57 67.31) (xy 118.11 67.31))
-    (stroke (width 0) (type default))
-  )
   (wire (pts (xy 128.27 54.61) (xy 129.54 54.61))
     (stroke (width 0) (type default))
@@
     (stroke (width 0) (type default))
   )
-  (wire (pts (xy 118.11 74.93) (xy 115.57 74.93))
-    (stroke (width 0) (type default))
-  )
   (wire (pts (xy 212.09 31.75) (xy 212.09 29.21))
     (stroke (width 0) (type default))
@@
     (stroke (width 0) (type default))
   )
-  (wire (pts (xy 118.11 67.31) (xy 118.11 69.85))
-    (stroke (width 0) (type default))
-  )
   (wire (pts (xy 168.91 53.34) (xy 170.18 53.34))
     (stroke (width 0) (type default))
@@
   )
   (wire (pts (xy 194.31 85.09) (xy 190.5 85.09))
-    (stroke (width 0) (type default))
-  )
-  (wire (pts (xy 118.11 72.39) (xy 118.11 74.93))
     (stroke (width 0) (type default))
   )
@@
     )
   )
-  (symbol (lib_id "Connector:USB_C_Receptacle_USB2.0") (at 100.33 69.85 0) (unit 1)
-    (in_bom yes) (on_board yes) (dnp no) (fields_autoplaced)
-    (property "Reference" "J3" (at 100.33 48.26 0)
-      (effects (font (size 1.27 1.27)))
-    )
-    (property "Value" "USB_C_Receptacle_USB2.0" (at 100.33 50.8 0)
-      (effects (font (size 1.27 1.27)))
-    )
-    (property "Footprint" "Connector_USB:USB_C_Receptacle_G-Switch_GT-USB-7010ASV" (at 104.14 69.85 0)
-      (effects (font (size 1.27 1.27)) hide)
-    )
-    (property "Datasheet" "https://www.usb.org/sites/default/files/documents/usb_type-c.zip" (at 104.14 69.85 0)
-      (effects (font (size 1.27 1.27)) hide)
-    )
-    (pin "A1")
-    (pin "A12")
-    (pin "A4")
-    (pin "A5")
-    (pin "A6")
-    (pin "A7")
-    (pin "A8")
-    (pin "A9")
-    (pin "B1")
-    (pin "B12")
-    (pin "B4")
-    (pin "B5")
-    (pin "B6")
-    (pin "B7")
-    (pin "B8")
-    (pin "B9")
-    (pin "S1")
-    (instances
-      (project "space-berry"
-        (path "/93269f17-932e-47e4-8e03-ce157f57b85f/2166ed60-c589-413b-a298-140af16eae77"
-          (reference "J3") (unit 1)
-        )
-        (path "/93269f17-932e-47e4-8e03-ce157f57b85f/b09b43d6-0155-4d95-82ac-b05a455defee"
-          (reference "J1") (unit 1)
-        )
-      )
-    )
-  )
   (symbol (lib_id "Device:C") (at 83.82 120.65 0) (unit 1)
     (in_bom yes) (on_board yes) (dnp no) (fields_autoplaced)
@@
         )
       )
-    )
-  )
-  (symbol (lib_id "power:GND") (at 96.52 96.52 0) (unit 1)
-    (in_bom yes) (on_board yes) (dnp no) (fields_autoplaced)
-    (property "Reference" "#PWR067" (at 96.52 102.87 0)
-      (effects (font (size 1.27 1.27)) hide)
-    )
-    (property "Value" "GND" (at 96.52 101.6 0)
-      (effects (font (size 1.27 1.27)))
-    )
-    (property "Footprint" "" (at 96.52 96.52 0)
-      (effects (font (size 1.27 1.27)) hide)
-    )
-    (property "Datasheet" "" (at 96.52 96.52 0)
-      (effects (font (size 1.27 1.27)) hide)
-    )
-    (pin "1")
-    (instances
-      (project "space-berry"
-        (path "/93269f17-932e-47e4-8e03-ce157f57b85f/2166ed60-c589-413b-a298-140af16eae77"
-          (reference "#PWR067") (unit 1)
-        )
-        (path "/93269f17-932e-47e4-8e03-ce157f57b85f/b09b43d6-0155-4d95-82ac-b05a455defee"
-          (reference "#PWR068") (unit 1)
-        )
-      )
